File: pcb/SX1303.kicad_sch (KiCad schematic)
At the start: 46 parts, among them U6 SX1303

Commit message: added:sch
Connections:
- net CONFIG_OK: now also U6.15 (GND); no longer U6.66 (GPIO[0])
- net GND: now also U6.11 (RADIO_CTRL[1]), U6.23 (VCC_CORE), U6.26 (RADIO_CTRL[7]), U6.32 (RADIO_B_IQ[3]), U6.4 (HOST_SCK), U6.41 (RADIO_A_IQ[3]), U6.42 (RADIO_A_MISO), U6.56 (VCC_CORE), U6.63 (GPIO[2]); no longer U6.15 (GND), U6.24 (GND), U6.25 (GND), U6.39 (GND), U6.46 (GND), U6.55 (GND), U6.6 (GND), U6.62 (GND), U6.9 (GND)
- net GPIO(10): now also U6.68 (RADIO_A_CSN); no longer U6.51 (GPIO[10])
- net GPIO(11): now also U6.67 (RADIO_A_MOSI); no longer U6.50 (GPIO[11])
- net GPIO(6): now also U6.6 (GND); no longer U6.57 (GPIO[6])
- net GPIO(9): now also U6.1 (HOST_CSN); no longer U6.52 (GPIO[9])
- net HOST_CSN: now also U6.18 (RADIO_B_CSN); no longer U6.1 (HOST_CSN)
- net HOST_MOSI: now also U6.20 (SP_VALID); no longer U6.3 (HOST_MOSI)
- net HOST_SCK: now also U6.21 (RADIO_B_SCK); no longer U6.4 (HOST_SCK)
- net PPS: now also U6.25 (GND); no longer U6.8 (PPS)
- net RADIO_A_CSN: no longer U6.68 (RADIO_A_CSN)
- net RADIO_A_MISO: now also U6.59 (GPIO[4]); no longer U6.42 (RADIO_A_MISO)
- net RADIO_A_MOSI: now also U6.16 (RADIO_CTRL[4]); no longer U6.67 (RADIO_A_MOSI)
- net RADIO_A_NRESET: now also U6.30 (VCC_IO); no longer U6.13 (RADIO_CTRL[3])
- net RADIO_A_SCK: now also U6.14 (VCC_IO); no longer U6.65 (RADIO_A_SCK)
- net RADIO_B_CSN: now also U6.35 (RADIO_B_IQ[0]); no longer U6.18 (RADIO_B_CSN)
- net RADIO_B_MISO: now also U6.50 (GPIO[11]); no longer U6.33 (RADIO_B_MISO)
- net RADIO_B_MOSI: now also U6.36 (RADIO_B_IQ[1]); no longer U6.19 (RADIO_B_MOSI)
- net RADIO_B_NRESET: now also U6.45 (RADIO_A_IQ[1]); no longer U6.28 (RADIO_CTRL[9])
- net RADIO_B_SCK: now also U6.38 (RADIO_B_IQ[2]); no longer U6.21 (RADIO_B_SCK)
- net RADIO_CTRL_(1): now also U6.28 (RADIO_CTRL[9]); no longer U6.11 (RADIO_CTRL[1])
- net RX_ON: now also U6.8 (PPS); no longer U6.59 (GPIO[4])
- net SX1261_DIO1: now also U6.3 (HOST_MOSI); no longer U6.54 (GPIO[7])
- net SX1302_CSD: now also U6.27 (RADIO_CTRL[8]); no longer U6.10 (RADIO_CTRL[0])
- net SX1302_GPIO_8: now also U6.2 (HOST_MISO); no longer U6.53 (GPIO[8])
- net SX1302_PA_ON: now also U6.33 (RADIO_B_MISO); no longer U6.16 (RADIO_CTRL[4])
- net SX1302_PS_EN: no longer U6.17 (RADIO_CTRL[5])
- net SX1302_RESET: now also U6.24 (GND); no longer U6.7 (RESET)
- net SX1302_RXTX_SW: now also U6.29 (RADIO_CTRL[10]); no longer U6.12 (RADIO_CTRL[2])
- net TX_ON: now also U6.12 (RADIO_CTRL[2]); no longer U6.63 (GPIO[2])
- net VCCCORE12: now also U6.22 (RADIO_CTRL[6]), U6.57 (GPIO[6]); no longer U6.23 (VCC_CORE), U6.56 (VCC_CORE)
- net VCCIO33: now also U6.10 (RADIO_CTRL[0]), U6.31 (RADIO_CTRL[11]), U6.64 (GPIO[1]); no longer U6.14 (VCC_IO), U6.30 (VCC_IO), U6.61 (VCC_IO)
- net at R17.2: now also U6.49 (RADIO_A_IQ[2]); no longer U6.32 (RADIO_B_IQ[3])
- net at R16.2: now also U6.37 (RADIO_B_IQ[4]); no longer U6.20 (SP_VALID)
- net at R19.1: now also U6.66 (GPIO[0]); no longer U6.49 (RADIO_A_IQ[2])
- net at R23.1: now also U6.60 (GPIO[3]); no longer U6.43 (RADIO_A_CLK_I)
- net at R25.1: now also U6.55 (GND); no longer U6.38 (RADIO_B_IQ[2])
- net at R28.1: now also U6.52 (GPIO[9]); no longer U6.35 (RADIO_B_IQ[0])
- net at TP2.1 (pin): now also U6.13 (RADIO_CTRL[3]); no longer U6.64 (GPIO[1])
- net at R18.2: now also U6.51 (GPIO[10]); no longer U6.34 (RADIO_B_CLK_I)
- net at R27.1: now also U6.53 (GPIO[8]); no longer U6.36 (RADIO_B_IQ[1])
- net at R14.1: now also U6.19 (RADIO_B_MOSI); no longer U6.2 (HOST_MISO)
- net at R26.1: now also U6.54 (GPIO[7]); no longer U6.37 (RADIO_B_IQ[4])
- net at R24.1: now also U6.58 (GPIO[5]); no longer U6.41 (RADIO_A_IQ[3])
- net at U6.44 (RADIO_A_IQ[0]): no longer R22.1
- net at R21.1: now also U6.62 (GND); no longer U6.45 (RADIO_A_IQ[1])
- net at U6.48 (RADIO_A_IQ[4]): no longer R20.1
- net at TP4.1 (pin): now also U6.7 (RESET); no longer U6.58 (GPIO[5])
- net at TP3.1 (pin): now also U6.9 (GND); no longer U6.60 (GPIO[3])
- new net: R22.1, U6.61 (VCC_IO)
- new net: R20.1, U6.65 (RADIO_A_SCK)
Other:
- moved on the sheet: U6
Changed lines of the file:
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@@
     )
   )
-  (symbol (lib_id "LoRa_PCIe_GW-rescue:SX1303") (at 185.42 149.86 0) (unit 1)
+  (symbol (lib_id "LoRa_PCIe_GW-rescue:SX1303") (at 185.42 149.86 270) (unit 1)
     (in_bom yes) (on_board yes) (dnp no)
-    (property "Reference" "U6" (at 247.269 91.2368 0)
+    (property "Reference" "U6" (at 244.0432 211.709 0)
       (effects (font (size 1.524 1.524)) (justify left bottom))
     )
-    (property "Value" "SX1303" (at 247.269 211.2264 0)
+    (property "Value" "SX1303" (at 124.0536 211.709 0)
       (effects (font (size 1.524 1.524)) (justify left bottom))
     )
-    (property "Footprint" "LoRa_PCIe_GW:vqfn68_7x7mm" (at 247.269 211.2264 0)
+    (property "Footprint" "LoRa_PCIe_GW:vqfn68_7x7mm" (at 124.0536 211.709 0)
       (effects (font (size 1.524 1.524)) hide)
     )
-    (property "Datasheet" "https://semtech.my.salesforce.com/sfc/p/#E0000000JelG/a/2R000000Hlli/Te0cB6.fNWAPfxRfoFz38R6LOTf3sLAJhD4CpS2RwFc" (at 247.269 211.2264 0)
+    (property "Datasheet" "https://semtech.my.salesforce.com/sfc/p/#E0000000JelG/a/2R000000Hlli/Te0cB6.fNWAPfxRfoFz38R6LOTf3sLAJhD4CpS2RwFc" (at 124.0536 211.709 0)
       (effects (font (size 1.524 1.524)) hide)
     )
